File: V3.kicad_pcb (KiCad board)
At the start: 2 copper layers, 30 parts, among them J1 USB_B, J2 Conn_01x02, J3 47219-2001, J4 MAX9814, J5 OLED, J6 Heartbeat, Q1 AO3401A, Q3 BSD840NH6327XTSA1, U1 AP9101CK-CMTRG1, U2 AMS1117-3.3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

Commit message: Finalise schematic and start routing
Parts:
- removed TP2: TP_Battery+, TestPoint:TestPoint_Pad_D1.0mm
- removed TP4: TP_Battery-, TestPoint:TestPoint_Pad_D1.0mm
- added R8: 45K, Resistor_SMD:R_1206_3216Metric, F.Cu at (141.8, 124.6)
- added REF**: MountingHole_2.7mm_M2.5, MountingHole:MountingHole_2.7mm_M2.5, F.Cu at (140.6, 138.6)
- added REF**: MountingHole_2.7mm_M2.5, MountingHole:MountingHole_2.7mm_M2.5, F.Cu at (106.6, 138.6)
- added REF**: MountingHole_2.7mm_M2.5, MountingHole:MountingHole_2.7mm_M2.5, F.Cu at (106.6, 104.6)
- C1, C2: value 100uF -> 1uF; footprint Capacitor_SMD:C_1812_4532Metric -> Capacitor_SMD:C_1206_3216Metric
- U2: value AMS1117-3.3 -> XC6222B331MR-G; footprint Package_TO_SOT_SMD:SOT-223-3_TabPin2 -> Package_TO_SOT_SMD:SOT-23-5
- moved TP3 51.8 mm to (110.6, 102.6)
- moved J2 43.5 mm to (106.6, 111.9), turned to 0 degrees
- moved R3 42.2 mm to (106.4, 117.8), turned to 180 degrees
- moved Q1 35.2 mm to (110.2, 110.8), turned to 180 degrees
- moved U1 33.2 mm to (111.2, 115.2), turned to 180 degrees
- moved J4 32.4 mm to (135.0, 132.6), turned to 0 degrees
- moved J6 31.4 mm to (121.4, 131.4), turned to 90 degrees
- moved Q3 30.4 mm to (115.6, 115.4), turned to 0 degrees
- moved TP1 30.1 mm to (118.0, 139.4)
- moved 3v3 27.8 mm to (113.0, 139.4)
- moved R2 26.6 mm to (114.4, 118.6), turned to 180 degrees
- moved C3 26.3 mm to (140.4, 132.4), turned to 0 degrees
- moved R1 25.2 mm to (121.0, 138.0)
- moved R5 25.2 mm to (136.4, 129.2), turned to 180 degrees
- moved J1 22.4 mm to (128.0, 137.6), turned to 0 degrees
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- renumbered TP5 to 3v3
Connections:
- U2 pad 1: GND -> VCC
- U2 pad 2: +3V3 -> GND
- U3 pad 21: unconnected-(U3-Pad21) -> Net-(U3-Pad21)
Routing:
- net VBUS: track 0.00 -> 55.7 mm
- net /FSPI_MOSI: track 0.00 -> 21.6 mm
- net /FSPICS0: track 0.00 -> 20.5 mm
- net /FSPI_CLK: track 0.00 -> 18.6 mm
- net VCC: track 0.00 -> 15.6 mm
- net +3V3: track 0.00 -> 13.0 mm, vias 0 -> 3
- net /USB_D-: track 0.00 -> 12.5 mm
- net /USB_D+: track 0.00 -> 12.5 mm
- net /FSPI_MISO: track 0.00 -> 12.2 mm
- net GND: track 6.90 -> 18.4 mm, vias 0 -> 9
- net Net-(Q3-Pad5): track 2.58 -> 11.4 mm
- net +BATT: track 3.25 -> 10.7 mm
- net -BATT: track 3.36 -> 8.93 mm
- net Net-(R4-Pad1): track 0.00 -> 3.69 mm
- net Net-(Q3-Pad2): track 5.64 -> 2.79 mm
Other:
- board outline added: 40 x 40 mm

Commit message: Route power
Parts:
- moved 3v3 36.9 mm to (110.4, 102.6)
- moved TP3 8.64 mm to (104.8, 109.0)
- moved C4 0.40 mm to (118.4, 116.6)
Routing:
- net +3V3: track 13.0 -> 82.7 mm, vias 3 -> 30
- net /SCL: track 0.00 -> 21.9 mm
- net /SDA: track 0.00 -> 20.7 mm
- net /MIC: track 0.00 -> 17.7 mm, vias 0 -> 1
- net Net-(U3-Pad21): track 0.00 -> 14.0 mm
- net +3.3VA: track 0.00 -> 9.56 mm
- net VCC: track 15.6 -> 21.1 mm
- net VBUS: track 55.7 -> 54.5 mm
- net GND: track 18.4 -> 18.3 mm, vias 9 -> 274
- added copper zone on B.Cu, net +3V3
- added copper zone on F.Cu, net +3V3

Commit message: Finish routing and export gerbers
Parts:
- added R10: 4.7K, Resistor_SMD:R_1206_3216Metric, F.Cu at (117.6, 137.1)
- added R9: 4.7K, Resistor_SMD:R_1206_3216Metric, F.Cu at (121.3, 135.7)
- added U5: USBLC6-2SC6, Package_TO_SOT_SMD:SOT-23-6, F.Cu at (132.6, 129.1)
- moved R1 9.09 mm to (112.0, 137.1), turned to 0 degrees
- moved R5 4.03 mm to (140.4, 129.7), turned to 0 degrees
- moved 3v3A 3.60 mm to (136.8, 129.3)
- moved C3 0.60 mm to (140.4, 133.0)
- moved REF** 0.14 mm to (140.7, 138.7)
- renumbered TP6 to 3v3A, TP1 to VBUS, TP3 to VCC
Connections:
- J1 pad 2: /USB_D- -> /USB_CONN_D-
- J1 pad 3: /USB_D+ -> /USB_CONN_D+
Routing:
- net +3V3: track 82.7 -> 125.3 mm, vias 30 -> 26
- net /SCL: track 21.9 -> 34.2 mm
- net VBUS: track 54.5 -> 66.0 mm
- net /USB_D-: track 12.5 -> 2.49 mm
- net /USB_D+: track 12.5 -> 2.66 mm
- net GND: track 18.3 -> 27.2 mm, vias 274 -> 287
- net /SDA: track 20.7 -> 29.4 mm
- net /USB_CONN_D+: track 0.00 -> 8.60 mm
- net /USB_CONN_D-: track 0.00 -> 7.30 mm
- net Net-(C4-Pad1): track 0.00 -> 5.78 mm, vias 0 -> 2
- net Net-(R7-Pad1): track 0.00 -> 5.55 mm
- net Net-(R6-Pad1): track 0.00 -> 3.54 mm
- net /ACCEL_INT2: track 0.00 -> 2.97 mm
- net /ACCEL_INT1: track 0.00 -> 2.34 mm
- net /MIC: track 17.7 -> 19.1 mm
- added copper zone on B.Cu, net GND
- added copper zone on F.Cu, net GND
Other:
- outline, holes or cut-outs redrawn

Commit message: Add 3d models, pcb & schematic touch up, graphics, update gerbers and add step file
Parts:
- added REF**: KiCad-Logo2_5mm_SilkScreen, Symbol:KiCad-Logo2_5mm_SilkScreen, B.Cu at (140.1, 129.6)
- added REF**: WEEE-Logo_4.2x6mm_SilkScreen, Symbol:WEEE-Logo_4.2x6mm_SilkScreen, B.Cu at (127.8, 135.2)
Routing:
- net +3V3: track 125.3 -> 123.8 mm
- net GND: vias 287 -> 263
Other:
- board text added: "Designed & assembled in Enschede by PintApple."
- board text added: "Team members: Bob Aaldering Julia Aalbers Marnix Laar Nian Luisman Irene Noorman Camiel Verdult"

Commit message: Switch out micro USB for USB-C
Parts:
- removed 3v3: TP_3v3, TestPoint:TestPoint_Pad_D1.0mm
- removed 3v3A: TP_3v3_Analog, TestPoint:TestPoint_Pad_D1.0mm
- added R11: 4.7K, Resistor_SMD:R_1206_3216Metric, F.Cu at (134.3, 136.9)
- added R12: 4.7K, Resistor_SMD:R_1206_3216Metric, F.Cu at (119.7, 139.7)
- added R13: 100, Resistor_SMD:R_1206_3216Metric, F.Cu at (133.1, 130.6)
- added R14: 100, Resistor_SMD:R_1206_3216Metric, F.Cu at (134.3, 128.2)
- added TP3: TP_3.3VA, TestPoint:TestPoint_Pad_D1.0mm, F.Cu at (110.5, 102.6)
- J1: value USB_B -> USB_C_Plug_USB2.0; footprint Connector_USB:USB_Micro-B_Wuerth_629105150521 -> Connector_USB:USB_C_Receptacle_GCT_USB4085
- R5: value 10K -> 100
- moved U5 5.71 mm to (138.3, 128.8)
- moved J1 4.04 mm to (124.9, 135.1)
- moved R5 2.51 mm to (141.2, 132.1)
- moved TP1 2.50 mm to (115.5, 139.4)
- moved J4 2.00 mm to (137.0, 132.6)
- moved C3 1.59 mm to (141.2, 134.4)
- renumbered VBUS to TP1, VCC to TP2
Connections:
- U5 pad 1: /USB_D+ -> Net-(R13-Pad2)
- U5 pad 3: /USB_D- -> Net-(R14-Pad2)
- U5 pad 4: /USB_CONN_D- -> /USB_CONN_D+
- U5 pad 6: /USB_CONN_D+ -> /USB_CONN_D-
Routing:
- net GND: track 27.2 -> 0.00 mm, vias 263 -> 29
- net VBUS: track 66.0 -> 84.5 mm
- net Net-(J1-PadA5): track 0.00 -> 12.2 mm, vias 0 -> 1
- net Net-(J1-PadB5): track 0.00 -> 10.0 mm, vias 0 -> 1
- net Net-(R13-Pad2): track 0.00 -> 6.38 mm
- net /USB_CONN_D-: track 7.30 -> 13.6 mm
- net +3.3VA: track 9.70 -> 4.95 mm
- net /USB_CONN_D+: track 8.60 -> 12.5 mm
- net /USB_D-: track 2.49 -> 5.06 mm
- net /MIC: track 19.1 -> 21.6 mm
- net Net-(R14-Pad2): track 0.00 -> 2.46 mm
- net +3V3: track 123.8 -> 125.3 mm, vias 26 -> 14
- net /USB_D+: track 2.66 -> 3.54 mm

Commit message: Add USB-C port
Parts:
- added C5: 100nF, Capacitor_SMD:C_1206_3216Metric, F.Cu at (141.5, 105.5)
- added R15: 1M, Resistor_SMD:R_1206_3216Metric, F.Cu at (112.0, 139.4)
- C1, C2: value 1uF -> 22uF
- J1: value USB_C_Plug_USB2.0 -> DX07S016JA1R1500; footprint Connector_USB:USB_C_Receptacle_GCT_USB4085 -> Footprints:JAE_DX07S016JA1R1500
- moved U5 5.80 mm to (132.5, 128.9)
- moved R14 4.47 mm to (132.9, 132.4)
- moved R13 4.38 mm to (137.3, 129.5)
- moved R6 3.50 mm to (141.5, 110.5)
- moved J1 3.39 mm to (127.9, 136.6)
- moved R7 2.74 mm to (141.5, 115.5)
Connections:
- net Net-(R6-Pad1) renamed /EN
- J1 pad S1: GND -> Net-(J1-PadS1)
- R11 pad 2: Net-(J1-PadB5) -> Net-(R11-Pad2)
- R12 pad 2: Net-(J1-PadA5) -> Net-(R12-Pad2)
- R13 pad 1: /USB_D- -> Net-(U5-Pad6)
- R13 pad 2: Net-(R13-Pad2) -> /USB_CONN_D-
- R14 pad 1: /USB_D+ -> /USB_CONN_D+
- U5 pad 1: Net-(R13-Pad2) -> /USB_D-
- U5 pad 3: Net-(R14-Pad2) -> /USB_D+
- U5 pad 4: /USB_CONN_D+ -> Net-(R14-Pad2)
- U5 pad 6: /USB_CONN_D- -> Net-(U5-Pad6)
Routing:
- net Net-(J1-PadS1): track 0.00 -> 47.5 mm, vias 0 -> 1
- net Net-(R12-Pad2): track 0.00 -> 12.5 mm, vias 0 -> 2
- net Net-(J1-PadA5): track 12.2 -> 0.00 mm, vias 1 -> 0
- net VBUS: track 84.5 -> 74.3 mm
- net Net-(R11-Pad2): track 0.00 -> 10.0 mm, vias 0 -> 2
- net Net-(J1-PadB5): track 10.0 -> 0.00 mm, vias 1 -> 0
- net Net-(R13-Pad2): track 6.38 -> 0.00 mm
- net /USB_CONN_D+: track 12.5 -> 6.60 mm
- net /USB_CONN_D-: track 13.6 -> 17.0 mm
- net +3V3: track 125.3 -> 122.0 mm
- net /EN: track 3.54 -> 6.31 mm
- net Net-(R7-Pad1): track 5.55 -> 8.25 mm
- net Net-(U5-Pad6): track 0.00 -> 2.61 mm
- net /MIC: track 21.6 -> 19.8 mm
- net Net-(R14-Pad2): track 2.46 -> 3.98 mm
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