File: V3.kicad_pcb (KiCad board)
At the start: 2 copper layers, 40 x 40 mm, 42 parts, among them J1 DX07S016JA1R1500, J2 Conn_01x02, J3 47219-2001, J4 MAX9814, J5 OLED, J6 Heartbeat, Q1 AO3401A, Q3 BSD840NH6327XTSA1, U1 AP9101CK-CMTRG1, U2 XC6222B331MR-G, U3 ESP32-S2-WROVER, U4 MMA8652FCR1, U5 USBLC6-2SC6

Commit message: Ja
Parts:
- removed REF** (x3): MountingHole_2.7mm_M2.5, MountingHole:MountingHole_2.7mm_M2.5
- removed REF**: KiCad-Logo2_5mm_SilkScreen, Symbol:KiCad-Logo2_5mm_SilkScreen
- removed REF**: WEEE-Logo_4.2x6mm_SilkScreen, Symbol:WEEE-Logo_4.2x6mm_SilkScreen
- removed U5: USBLC6-2SC6, Package_TO_SOT_SMD:SOT-23-6
- added H1: MountingHole_Pad, MountingHole:MountingHole_2.2mm_M2_Pad, F.Cu at (106.5, 104.5)
- added H2: MountingHole_Pad, MountingHole:MountingHole_2.2mm_M2_Pad, F.Cu at (106.5, 138.5)
- added H3: MountingHole_Pad, MountingHole:MountingHole_2.2mm_M2_Pad, F.Cu at (140.5, 138.5)
- added R16: 2.7K, Resistor_SMD:R_1206_3216Metric, F.Cu at (138.0, 129.0)
- added R17: 10K, Resistor_SMD:R_1206_3216Metric, F.Cu at (141.4, 128.5)
- Q1: value AO3401A -> BSH201,215
- R3: renamed from R12; value 4.7K -> 5.1K
- R4: renamed from R11; value 4.7K -> 5.1K
- moved R1 3.20 mm to (131.8, 129.4), turned to 90 degrees
- moved R2 3.10 mm to (134.2, 129.4), turned to -90 degrees
- moved R10 1.10 mm to (141.8, 123.5)
- moved R5 0.90 mm to (112.0, 136.2)
- turned R3 to 180 degrees
- renumbered TP3 to 3v3, C5 to C4, C4 to C5, Q3 to Q2, R14 to R1, R8 to R10, R6 to R11, R9 to R12, R10 to R13, R4 to R14, R7 to R15, R13 to R2, R1 to R5, R2 to R6, R15 to R7, R3 to R8, R5 to R9, TP1 to VBUS, TP2 to VCC
Connections:
- J1 pad 3: Net-(R12-Pad2) -> Net-(J1-Pad3)
- R1 pad 1: /USB_CONN_D+ -> /USB_CONN_D-
- R1 pad 2: Net-(R14-Pad2) -> /USB_D-
- R2 pad 1: Net-(U5-Pad6) -> /USB_D+
- R2 pad 2: /USB_CONN_D- -> /USB_CONN_D+
- R3 pad 1: GND -> Net-(J1-Pad3)
- R3 pad 2: Net-(R12-Pad2) -> GND
- U3 pad 25: unconnected-(U3-Pad25) -> Net-(R16-Pad1)
Routing:
- net +BATT: track 10.7 -> 53.1 mm, vias 0 -> 2
- net Net-(R12-Pad2): track 12.5 -> 0.00 mm, vias 2 -> 0
- net Net-(J1-Pad3): track 0.00 -> 12.5 mm, vias 0 -> 2
- net VBUS: track 74.3 -> 61.9 mm
- net Net-(R16-Pad1): track 0.00 -> 8.99 mm
- net /USB_CONN_D-: track 17.0 -> 9.38 mm
- net /USB_CONN_D+: track 6.60 -> 11.2 mm
- net Net-(R14-Pad2): track 3.98 -> 0.00 mm
- net /USB_D-: track 6.16 -> 2.53 mm
- net Net-(U5-Pad6): track 2.61 -> 0.00 mm
- net /USB_D+: track 2.24 -> 3.19 mm
- net +3V3: track 122.0 -> 122.8 mm, vias 14 -> 13
- net Net-(R10-Pad1): track 14.0 -> 14.7 mm
- net GND: vias 48 -> 37

Commit message: v3.1
Parts:
- removed VBUS: TP_VBUS, TestPoint:TestPoint_Pad_D1.0mm
- added SW1: BUTTON, Button_Switch_SMD:SW_Push_1P1T_NO_CK_KSC6xxJ, F.Cu at (118.2, 139.0)
- R12, R13: moved to B.Cu
- TP2: renamed from VCC; value TP_VCC -> VCC
- TP3: renamed from 3v3; value TP_3.3VA -> 3v3
- moved R3 14.8 mm to (134.4, 138.6), turned to 90 degrees
- moved R4 4.36 mm to (133.0, 132.8), turned to 180 degrees
- moved R12 4.04 mm to (117.4, 134.6), turned to 180 degrees
- moved R6 3.20 mm to (111.2, 118.6), turned to 0 degrees
- moved R5 3.03 mm to (112.4, 139.2), turned to 90 degrees
- moved R7 1.77 mm to (110.2, 139.2), turned to -90 degrees
- moved C5 0.63 mm to (118.6, 116.0)
- moved R10 0.40 mm to (141.4, 123.5)
- moved R13 0.22 mm to (117.4, 137.0)
Connections:
- U3 pad 17: unconnected-(U3-Pad17) -> Net-(SW1-Pad2)
Routing:
- net Net-(SW1-Pad2): track 0.00 -> 20.4 mm
- net +3V3: track 122.8 -> 129.8 mm, vias 13 -> 14
- net Net-(J1-Pad9): track 10.0 -> 3.78 mm, vias 2 -> 0
- net Net-(Q2-Pad5): track 11.4 -> 8.18 mm, vias 0 -> 2
- net /SDA: track 29.4 -> 32.3 mm
- net VBUS: track 61.9 -> 59.3 mm
- net Net-(J1-PadS1): track 47.5 -> 46.2 mm
- net Net-(J1-Pad3): track 12.5 -> 11.6 mm
- net Net-(C5-Pad1): track 5.78 -> 5.01 mm
- net /SCL: track 34.5 -> 35.2 mm
- net /USB_CONN_D-: track 9.38 -> 8.87 mm
- net GND: vias 37 -> 33
