File: V3.kicad_sch (KiCad schematic)
At the start: 37 parts, among them J1 DX07S016JA1R1500, J2 Conn_01x02, J3 47219-2001, J4 MAX9814, J5 OLED, J6 Heartbeat, Q1 AO3401A, Q3 BSD840NH6327XTSA1, U1 AP9101CK-CMTRG1, U2 XC6222B331MR-G, U3 ESP32-S2-WROVER, U4 MMA8652FCR1, U5 USBLC6-2SC6

Commit message: Ja
Parts:
- removed U5: USBLC6-2SC6, Package_TO_SOT_SMD:SOT-23-6, symbol Power_Protection:USBLC6-2SC6
- added H1, H2, H3: MountingHole_Pad, MountingHole:MountingHole_2.2mm_M2_Pad, symbol Mechanical:MountingHole_Pad
- added R16: 2.7K, Resistor_SMD:R_1206_3216Metric, symbol Device:R_Small
- added R17: 10K, Resistor_SMD:R_1206_3216Metric, symbol Device:R_Small
- Q1: value AO3401A -> BSH201,215
- R3: renamed from R12; value 4.7K -> 5.1K
- R4: renamed from R11; value 4.7K -> 5.1K
- renumbered C5 to C4, C4 to C5, Q3 to Q2, R14 to R1, R8 to R10, R6 to R11, R9 to R12, R10 to R13, R4 to R14, R7 to R15, R13 to R2, R1 to R5, R2 to R6, R15 to R7, R3 to R8, R5 to R9
Connections:
- net +BATT: now also R16.2
- net GND: now also R3.2, H1.1, H2.1, H3.1, R17.1; no longer R3.1
- net USB_CONN_D+: now also R2.2; no longer R1.1
- net USB_CONN_D-: now also R1.1; no longer R2.2
- net USB_D+: now also R2.1
- net USB_D-: now also R1.2
- net at J1.3 (CC1): now also R3.1; no longer R3.2
- net at U3.25 (IO26): now also R16.1, R17.2
Other:
- note added: "Simulation: https://tinyurl.com/yxeflho3"
- note added: "USB-C port"
- note removed: "Simulation: https://tinyurl.com/y7ddr9ho"
- note removed: "USB and ESD protection"
- moved on the sheet: R1, R2, R3, R4

Commit message: v3.1
Parts:
- removed TP1: TP_VBUS, TestPoint:TestPoint_Pad_D1.0mm, symbol Connector:TestPoint
- added SW1: BUTTON, Button_Switch_SMD:SW_Push_1P1T_NO_CK_KSC6xxJ, symbol Switch:SW_Push
- TP2: value TP_VCC -> VCC
- TP3: value TP_3.3VA -> 3v3
Connections:
- net +3V3: now also SW1.1
- net at U3.17 (IO14): now also SW1.2
